Commit message: Ouster Mesh updated

File: ouster_description/urdf/OS1-128.urdf.xacro (robot description, xacro)
@@ -18,5 +18,5 @@
       <visual>
         <geometry>
-          <mesh filename="package://ouster_description/meshes/HDL32E_base.dae" />
+          <mesh filename="package://ouster_description/meshes/OS1.dae" />
         </geometry>
       </visual>
@@ -42,5 +42,5 @@
         <origin xyz="0 0 -0.09081" rpy="0 0 0" />
         <geometry>
-          <mesh filename="package://ouster_description/meshes/HDL32E_scan.dae" />
+          <mesh filename="package://ouster_description/meshes/OS1.dae" />
         </geometry>
       </visual>
