Commit message: added 4 ouster, camera and updated world models

File: husky_description/urdf/accessories/flir_blackfly_mount.urdf.xacro (robot description, xacro)
@@ -2,4 +2,5 @@
 <robot xmlns:xacro="http://ros.org/wiki/xacro">
   <xacro:include filename="$(find fath_pivot_mount_description)/urdf/lockmount.urdf.xacro"/>
+  <!-- Using local flir_camera_description package instead of the one from the ROS distribution. -->
   <xacro:include filename="$(find flir_camera_description)/urdf/flir_blackflys.urdf.xacro"/>
   <xacro:macro name="flir_blackfly_mount" params="prefix:=blackfly

File: husky_description/urdf/husky.urdf.xacro (robot description, xacro)
@@ -70,18 +70,12 @@
   <xacro:arg name="laser_3d_secondary_rpy"        default="$(optenv HUSKY_LASER_3D_SECONDARY_RPY 0 0 -3.14159)" />
 <!-- Ouster LiDAR Primary and Secondary -->
-  <xacro:arg name="OUSTER_3D_enabled"              default="$(optenv HUSKY_OUSTER_3D_ENABLED 1)" />
-  <xacro:arg name="OUSTER_3D_topic"                default="$(optenv HUSKY_OUSTER_3D_TOPIC ouster_points)"/>
-  <xacro:arg name="OUSTER_3D_tower"                default="$(optenv HUSKY_OUSTER_3D_TOWER 1)"/>
-  <xacro:arg name="OUSTER_3D_prefix"               default="$(optenv HUSKY_OUSTER_3D_PREFIX )"/>
-  <xacro:arg name="OUSTER_3D_parent"               default="$(optenv HUSKY_OUSTER_3D_PARENT top_plate_link)"/>
-  <xacro:arg name="OUSTER_3D_xyz"                  default="$(optenv HUSKY_OUSTER_3D_XYZ 0 0 0)" />
-  <xacro:arg name="OUSTER_3D_rpy"                  default="$(optenv HUSKY_OUSTER_3D_RPY 0 0 0)" />
-  <xacro:arg name="OUSTER_3D_secondary_enabled"    default="$(optenv HUSKY_OUSTER_3D_SECONDARY_ENABLED 0)" />
-  <xacro:arg name="OUSTER_3D_secondary_topic"      default="$(optenv HUSKY_OUSTER_3D_SECONDARY_TOPIC ouster_secondary_points)"/>
-  <xacro:arg name="OUSTER_3D_secondary_tower"      default="$(optenv HUSKY_OUSTER_3D_SECONDARY_TOWER 1)"/>
-  <xacro:arg name="OUSTER_3D_secondary_prefix"     default="$(optenv HUSKY_OUSTER_3D_SECONDARY_PREFIX secondary_)"/>
-  <xacro:arg name="OUSTER_3D_secondary_parent"     default="$(optenv HUSKY_OUSTER_3D_SECONDARY_PARENT top_plate_link)"/>
-  <xacro:arg name="OUSTER_3D_secondary_xyz"        default="$(optenv HUSKY_OUSTER_3D_SECONDARY_XYZ 0 0 0)" />
-  <xacro:arg name="OUSTER_3D_secondary_rpy"        default="$(optenv HUSKY_OUSTER_3D_SECONDARY_RPY 0 0 -3.14159)" />
+  <!-- No LiDAR = 0
+  OS1 = 1
+  OS2 = 2
+  OS0 = 3
+  -->
+  <xacro:arg name="OUSTER_OS"              default="$(optenv HUSKY_OUSTER 0)" />
+  <!-- <xacro:arg name="OUSTER_OS2_enabled"              default="$(optenv HUSKY_OUSTER_OS2_ENABLED 0)" /> -->
+  <!-- <xacro:arg name="OUSTER_OS0_enabled"              default="$(optenv HUSKY_OUSTER_OS0_ENABLED 0)" /> -->
   <!-- Realsense Camera Primary and Secondary -->
   <xacro:arg name="realsense_enabled"             default="$(optenv HUSKY_REALSENSE_ENABLED 0)" />
@@ -105,11 +99,4 @@
   <xacro:arg name="blackfly_xyz"                      default="$(optenv HUSKY_BLACKFLY_XYZ 0 0 0)"/>
   <xacro:arg name="blackfly_rpy"                      default="$(optenv HUSKY_BLACKFLY_RPY 0 0 0)"/>
-  <xacro:arg name="blackfly_secondary_enabled"        default="$(optenv HUSKY_BLACKFLY_SECONDARY 0)"/>
-  <xacro:arg name="blackfly_secondary_mount_enabled"  default="$(optenv HUSKY_BLACKFLY_SECONDARY_MOUNT_ENABLED 1)"/>
-  <xacro:arg name="blackfly_secondary_mount_angle"    default="$(optenv HUSKY_BLACKFLY_SECONDARY_MOUNT_ANGLE 0)"/>
-  <xacro:arg name="blackfly_secondary_prefix"         default="$(optenv HUSKY_BLACKFLY_SECONDARY_PREFIX blackfly_secondary)"/>
-  <xacro:arg name="blackfly_secondary_parent"         default="$(optenv HUSKY_BLACKFLY_SECONDARY_PARENT top_plate_link)"/>
-  <xacro:arg name="blackfly_secondary_xyz"            default="$(optenv HUSKY_BLACKFLY_SECONDARY_XYZ 0 0 0)"/>
-  <xacro:arg name="blackfly_secondary_rpy"            default="$(optenv HUSKY_BLACKFLY_SECONDARY_RPY 0 0 0)"/>
   <!-- Bumper Extension -->
   <xacro:property name="husky_front_bumper_extend"  value="$(optenv HUSKY_FRONT_BUMPER_EXTEND 0)" />
@@ -134,11 +121,7 @@
   <xacro:include filename="$(find husky_description)/urdf/decorations.urdf.xacro" />
   <xacro:include filename="$(find husky_description)/urdf/wheel.urdf.xacro" />
-  <xacro:include filename="$(find ouster_description)/urdf/OS1-128.urdf.xacro"/>
-  <xacro:OS1-128 parent="top_plate_link" name="ouster" topic="/ouster_points" organize_cloud="false" hz="10" samples="2048" gpu="true">
-    <origin xyz="0 0 0.1" rpy="0 0 0" />
-  </xacro:OS1-128>
-  <!-- <xacro:include filename="$(find ouster_description)/urdf/OS1-64.urdf.xacro"/>
-  <xacro:OS1-128 parent="top_plate_link" name="ouster" topic="/ouster_points" organize_cloud="false" hz="10" samples="1024" gpu="true">
-    <origin xyz="0 0 0.1" rpy="0 0 0" />
+  <!-- <xacro:include filename="$(find ouster_description)/urdf/OS2-128.urdf.xacro"/>
+  <xacro:OS1-128 parent="top_plate_link" name="ouster">
+    <origin xyz="0 0 0.075" rpy="0 0 0" />
   </xacro:OS1-128> -->
   <xacro:property name="M_PI" value="3.14159"/>
@@ -284,12 +267,4 @@
     </xacro:flir_blackfly_mount>
   </xacro:if>
-  <xacro:if value="$(arg blackfly_secondary_enabled)">
-    <xacro:flir_blackfly_mount prefix="$(arg blackfly_secondary_prefix)"
-                                parent="$(arg blackfly_secondary_parent)"
-                                mount_enabled="$(arg blackfly_secondary_mount_enabled)"
-                                mount_angle="$(arg blackfly_secondary_mount_angle)">
-      <origin xyz="$(arg blackfly_secondary_xyz)" rpy="$(arg blackfly_secondary_rpy)"/>
-    </xacro:flir_blackfly_mount>
-  </xacro:if>
   <!--
     Velodyne 3D LiDAR Primary and Secondary
@@ -320,30 +295,31 @@
   </xacro:if>
   <!--
-    Ouster 3D LiDAR Primary and Secondary
-  -->
-  <!-- <xacro:if value="$(arg OUSTER_3D_enabled)">
-    <xacro:if value="$(arg OUSTER_3D_tower)">
-      <xacro:vlp16_mount prefix="$(arg OUSTER_3D_prefix)" parent_link="$(arg OUSTER_3D_parent)" topic="$(arg OUSTER_3D_topic)">
-        <origin xyz="$(arg OUSTER_3D_xyz)" rpy="$(arg OUSTER_3D_rpy)" />
-      </xacro:vlp16_mount>
-    </xacro:if>
-    <xacro:unless value="$(arg OUSTER_3D_tower)">
-      <xacro:VLP-16 parent="$(arg OUSTER_3D_parent)" topic="$(arg OUSTER_3D_topic)" name="$(arg OUSTER_3D_prefix)ouster">
-        <origin xyz="$(arg OUSTER_3D_xyz)" rpy="$(arg OUSTER_3D_rpy)" />
-      </xacro:VLP-16>
-    </xacro:unless>
-  </xacro:if>
-  <xacro:if value="$(arg OUSTER_3D_secondary_enabled)">
-    <xacro:if value="$(arg OUSTER_3D_secondary_tower)">
-      <xacro:vlp16_mount prefix="$(arg OUSTER_3D_secondary_prefix)" parent_link="$(arg OUSTER_3D_secondary_parent)" topic="$(arg OUSTER_3D_secondary_topic)">
-        <origin xyz="$(arg OUSTER_3D_secondary_xyz)" rpy="$(arg OUSTER_3D_secondary_rpy)" />
-      </xacro:vlp16_mount>
-    </xacro:if>
-    <xacro:unless value="$(arg OUSTER_3D_secondary_tower)">
-      <xacro:VLP-16 parent="$(arg OUSTER_3D_secondary_parent)" topic="$(arg OUSTER_3D_secondary_topic)" name="$(arg OUSTER_3D_secondary_prefix)ouster">
-        <origin xyz="$(arg OUSTER_3D_secondary_xyz)" rpy="$(arg OUSTER_3D_secondary_rpy)" />
-      </xacro:VLP-16>
-    </xacro:unless>
-  </xacro:if> -->
+    Ouster OS LiDAR
+  -->
+  <xacro:property name="model" value="$(arg OUSTER_OS)"/>
+  <xacro:if value="${model == 1}">
+    <xacro:include filename="$(find ouster_description)/urdf/OS1-128.urdf.xacro"/>
+    <xacro:OS1-128 parent="top_plate_link" name="ouster">
+      <origin xyz="0 0 0.075" rpy="0 0 0" />
+    </xacro:OS1-128>
+  </xacro:if>
+  <xacro:if value="${model == 2}">
+    <xacro:include filename="$(find ouster_description)/urdf/OS2-128.urdf.xacro"/>
+    <xacro:OS2-128 parent="top_plate_link" name="ouster">
+      <origin xyz="0 0 0.075" rpy="0 0 0" />
+    </xacro:OS2-128>
+  </xacro:if>
+  <xacro:if value="${model == 3}">
+    <xacro:include filename="$(find ouster_description)/urdf/OS0-128.urdf.xacro"/>
+    <xacro:OS0-128 parent="top_plate_link" name="ouster">
+      <origin xyz="0 0 0.075" rpy="0 0 0" />
+    </xacro:OS0-128>
+  </xacro:if>
+  <xacro:if value="${model == 4}">
+    <xacro:include filename="$(find ouster_description)/urdf/OSD-128.urdf.xacro"/>
+    <xacro:OSD-128 parent="top_plate_link" name="ouster">
+      <origin xyz="0 0 0.075" rpy="0 0 0" />
+    </xacro:OSD-128>
+  </xacro:if>
   <gazebo>
     <plugin name="gazebo_ros_control" filename="libgazebo_ros_control.so">

File: ouster_description/urdf/OS1-128.urdf.xacro (robot description, xacro)
@@ -2,5 +2,5 @@
 <robot xmlns:xacro="http://www.ros.org/wiki/xacro" name="OS1-128">
   <xacro:property name="M_PI" value="3.1415926535897931" />
-  <xacro:macro name="OS1-128" params="*origin parent:=base_link name:=ouster topic:=/ouster_points organize_cloud:=true hz:=10 lasers:=128 samples:=2048 collision_range:=0.3 min_range:=0.3 max_range:=100.0 noise:=0.008 min_angle:=-${M_PI} max_angle:=${M_PI} gpu:=false">
+  <xacro:macro name="OS1-128" params="*origin parent:=base_link name:=ouster topic:=/ouster_points organize_cloud:=true hz:=10 lasers:=128 samples:=2048 collision_range:=0.5 min_range:=0.5 max_range:=90.0 noise:=0.008 min_angle:=-${M_PI} max_angle:=${M_PI} gpu:=true">
     <joint name="${name}_base_mount_joint" type="fixed">
       <xacro:insert_block name="origin" />
