Commit message: added 27 ouster xacro and updated husky xacro

File: husky_description/urdf/husky.urdf copy.xacro (robot description, xacro)
@@ -305,160 +305,20 @@
   </xacro:if>
   <xacro:if value="${model == 2}">
-    <xacro:include filename="$(find ouster_description)/urdf/OS2-128-N1.urdf.xacro"/>
-    <xacro:OS2-128-N1 parent="top_plate_link" name="ouster">
+    <xacro:include filename="$(find ouster_description)/urdf/OS2-128.urdf.xacro"/>
+    <xacro:OS2-128 parent="top_plate_link" name="ouster">
       <origin xyz="0 0 0.075" rpy="0 0 0" />
-    </xacro:OS2-128-N1>
+    </xacro:OS2-128>
   </xacro:if>
   <xacro:if value="${model == 3}">
-    <xacro:include filename="$(find ouster_description)/urdf/OS0-128-N1.urdf.xacro"/>
-    <xacro:OS0-128-N1 parent="top_plate_link" name="ouster">
+    <xacro:include filename="$(find ouster_description)/urdf/OS0-128.urdf.xacro"/>
+    <xacro:OS0-128 parent="top_plate_link" name="ouster">
       <origin xyz="0 0 0.075" rpy="0 0 0" />
-    </xacro:OS0-128-N1>
+    </xacro:OS0-128>
   </xacro:if>
   <xacro:if value="${model == 4}">
-    <xacro:include filename="$(find ouster_description)/urdf/OS1-64-N1.urdf.xacro"/>
-    <xacro:OS1-64-N1 parent="top_plate_link" name="ouster">
+    <xacro:include filename="$(find ouster_description)/urdf/OSD-128.urdf.xacro"/>
+    <xacro:OSD-128 parent="top_plate_link" name="ouster">
       <origin xyz="0 0 0.075" rpy="0 0 0" />
-    </xacro:OS1-64-N1>
-  </xacro:if>
-  <xacro:if value="${model == 5}">
-    <xacro:include filename="$(find ouster_description)/urdf/OS2-64-N1.urdf.xacro"/>
-    <xacro:OS2-64-N1 parent="top_plate_link" name="ouster">
-      <origin xyz="0 0 0.075" rpy="0 0 0" />
-    </xacro:OS2-64-N1>
-  </xacro:if>
-  <xacro:if value="${model == 6}">
-    <xacro:include filename="$(find ouster_description)/urdf/OS0-64-N1.urdf.xacro"/>
-    <xacro:OS0-64-N1 parent="top_plate_link" name="ouster">
-      <origin xyz="0 0 0.075" rpy="0 0 0" />
-    </xacro:OS0-64-N1>
-  </xacro:if>
-  <xacro:if value="${model == 7}">
-    <xacro:include filename="$(find ouster_description)/urdf/OS1-32-N1.urdf.xacro"/>
-    <xacro:OS1-32-N1 parent="top_plate_link" name="ouster">
-      <origin xyz="0 0 0.075" rpy="0 0 0" />
-    </xacro:OS1-32-N1>
-  </xacro:if>
-  <xacro:if value="${model == 8}">
-    <xacro:include filename="$(find ouster_description)/urdf/OS2-32-N1.urdf.xacro"/>
-    <xacro:OS2-32-N1 parent="top_plate_link" name="ouster">
-      <origin xyz="0 0 0.075" rpy="0 0 0" />
-    </xacro:OS2-32-N1>
-  </xacro:if>
-  <xacro:if value="${model == 9}">
-    <xacro:include filename="$(find ouster_description)/urdf/OS0-32-N1.urdf.xacro"/>
-    <xacro:OS0-32-N1 parent="top_plate_link" name="ouster">
-      <origin xyz="0 0 0.075" rpy="0 0 0" />
-    </xacro:OS0-32-N1>
-  </xacro:if>
-  <xacro:property name="model" value="$(arg OUSTER_OS)"/>
-  <xacro:if value="${model == 10}">
-    <xacro:include filename="$(find ouster_description)/urdf/OS1-128-N2.urdf.xacro"/>
-    <xacro:OS1-128-N2 parent="top_plate_link" name="ouster">
-      <origin xyz="0 0 0.075" rpy="0 0 0" />
-    </xacro:OS1-128-N2>
-  </xacro:if>
-  <xacro:if value="${model == 11}">
-    <xacro:include filename="$(find ouster_description)/urdf/OS2-128-N2.urdf.xacro"/>
-    <xacro:OS2-128-N2 parent="top_plate_link" name="ouster">
-      <origin xyz="0 0 0.075" rpy="0 0 0" />
-    </xacro:OS2-128-N2>
-  </xacro:if>
-  <xacro:if value="${model == 12}">
-    <xacro:include filename="$(find ouster_description)/urdf/OS0-128-N2.urdf.xacro"/>
-    <xacro:OS0-128-N2 parent="top_plate_link" name="ouster">
-      <origin xyz="0 0 0.075" rpy="0 0 0" />
-    </xacro:OS0-128-N2>
-  </xacro:if>
-  <xacro:if value="${model == 13}">
-    <xacro:include filename="$(find ouster_description)/urdf/OS1-64-N2.urdf.xacro"/>
-    <xacro:OS1-64-N2 parent="top_plate_link" name="ouster">
-      <origin xyz="0 0 0.075" rpy="0 0 0" />
-    </xacro:OS1-64-N2>
-  </xacro:if>
-  <xacro:if value="${model == 14}">
-    <xacro:include filename="$(find ouster_description)/urdf/OS2-64-N2.urdf.xacro"/>
-    <xacro:OS2-64-N2 parent="top_plate_link" name="ouster">
-      <origin xyz="0 0 0.075" rpy="0 0 0" />
-    </xacro:OS2-64-N2>
-  </xacro:if>
-  <xacro:if value="${model == 15}">
-    <xacro:include filename="$(find ouster_description)/urdf/OS0-64-N2.urdf.xacro"/>
-    <xacro:OS0-64-N2 parent="top_plate_link" name="ouster">
-      <origin xyz="0 0 0.075" rpy="0 0 0" />
-    </xacro:OS0-64-N2>
-  </xacro:if>
-  <xacro:if value="${model == 16}">
-    <xacro:include filename="$(find ouster_description)/urdf/OS1-32-N2.urdf.xacro"/>
-    <xacro:OS1-32-N2 parent="top_plate_link" name="ouster">
-      <origin xyz="0 0 0.075" rpy="0 0 0" />
-    </xacro:OS1-32-N2>
-  </xacro:if>
-  <xacro:if value="${model == 17}">
-    <xacro:include filename="$(find ouster_description)/urdf/OS2-32-N2.urdf.xacro"/>
-    <xacro:OS2-32-N2 parent="top_plate_link" name="ouster">
-      <origin xyz="0 0 0.075" rpy="0 0 0" />
-    </xacro:OS2-32-N2>
-  </xacro:if>
-  <xacro:if value="${model == 18}">
-    <xacro:include filename="$(find ouster_description)/urdf/OS0-32-N2.urdf.xacro"/>
-    <xacro:OS0-32-N2 parent="top_plate_link" name="ouster">
-      <origin xyz="0 0 0.075" rpy="0 0 0" />
-    </xacro:OS0-32-N2>
-  </xacro:if>
-  <xacro:property name="model" value="$(arg OUSTER_OS)"/>
-  <xacro:if value="${model == 19}">
-    <xacro:include filename="$(find ouster_description)/urdf/OS1-128-N3.urdf.xacro"/>
-    <xacro:OS1-128-N3 parent="top_plate_link" name="ouster">
-      <origin xyz="0 0 0.075" rpy="0 0 0" />
-    </xacro:OS1-128-N3>
-  </xacro:if>
-  <xacro:if value="${model == 20}">
-    <xacro:include filename="$(find ouster_description)/urdf/OS2-128-N3.urdf.xacro"/>
-    <xacro:OS2-128-N3 parent="top_plate_link" name="ouster">
-      <origin xyz="0 0 0.075" rpy="0 0 0" />
-    </xacro:OS2-128-N3>
-  </xacro:if>
-  <xacro:if value="${model == 21}">
-    <xacro:include filename="$(find ouster_description)/urdf/OS0-128-N3.urdf.xacro"/>
-    <xacro:OS0-128-N3 parent="top_plate_link" name="ouster">
-      <origin xyz="0 0 0.075" rpy="0 0 0" />
-    </xacro:OS0-128-N3>
-  </xacro:if>
-  <xacro:if value="${model == 22}">
-    <xacro:include filename="$(find ouster_description)/urdf/OS1-64-N3.urdf.xacro"/>
-    <xacro:OS1-64-N3 parent="top_plate_link" name="ouster">
-      <origin xyz="0 0 0.075" rpy="0 0 0" />
-    </xacro:OS1-64-N3>
-  </xacro:if>
-  <xacro:if value="${model == 23}">
-    <xacro:include filename="$(find ouster_description)/urdf/OS2-64-N3.urdf.xacro"/>
-    <xacro:OS2-64-N3 parent="top_plate_link" name="ouster">
-      <origin xyz="0 0 0.075" rpy="0 0 0" />
-    </xacro:OS2-64-N3>
-  </xacro:if>
-  <xacro:if value="${model == 24}">
-    <xacro:include filename="$(find ouster_description)/urdf/OS0-64-N3.urdf.xacro"/>
-    <xacro:OS0-64-N3 parent="top_plate_link" name="ouster">
-      <origin xyz="0 0 0.075" rpy="0 0 0" />
-    </xacro:OS0-64-N3>
-  </xacro:if>
-  <xacro:if value="${model == 25}">
-    <xacro:include filename="$(find ouster_description)/urdf/OS1-32-N3.urdf.xacro"/>
-    <xacro:OS1-32-N3 parent="top_plate_link" name="ouster">
-      <origin xyz="0 0 0.075" rpy="0 0 0" />
-    </xacro:OS1-32-N3>
-  </xacro:if>
-  <xacro:if value="${model == 26}">
-    <xacro:include filename="$(find ouster_description)/urdf/OS2-32-N3.urdf.xacro"/>
-    <xacro:OS2-32-N3 parent="top_plate_link" name="ouster">
-      <origin xyz="0 0 0.075" rpy="0 0 0" />
-    </xacro:OS2-32-N3>
-  </xacro:if>
-  <xacro:if value="${model == 27}">
-    <xacro:include filename="$(find ouster_description)/urdf/OS0-32-N3.urdf.xacro"/>
-    <xacro:OS0-32-N3 parent="top_plate_link" name="ouster">
-      <origin xyz="0 0 0.075" rpy="0 0 0" />
-    </xacro:OS0-32-N3>
+    </xacro:OSD-128>
   </xacro:if>
   <gazebo>

File: ouster_description/urdf/OS1-32-N2.urdf.xacro (robot description, xacro)
@@ -1,8 +1,6 @@
 <?xml version="1.0"?>
-<robot xmlns:xacro="http://www.ros.org/wiki/xacro" name="OS1-128">
-<!-- <robot xmlns:xacro="http://www.ros.org/wiki/xacro" name="OS0-128"> -->
+<robot xmlns:xacro="http://www.ros.org/wiki/xacro" name="OS1-32-N2">
   <xacro:property name="M_PI" value="3.1415926535897931" />
-  <!-- <xacro:macro name="OS1-128" params="*origin parent:=base_link name:=ouster topic:=/ouster_points organize_cloud:=true hz:=10 lasers:=128 samples:=2048 collision_range:=0.5 min_range:=0.5 max_range:=35.0 noise:=0.008 min_angle:=-${M_PI} max_angle:=${M_PI} gpu:=true"> -->
-    <xacro:macro name="OS0-128" params="*origin parent:=base_link name:=ouster topic:=/ouster_points organize_cloud:=true hz:=10 lasers:=128 samples:=2048 collision_range:=0.5 min_range:=0.5 max_range:=35.0 noise:=0.008 min_angle:=-${M_PI} max_angle:=${M_PI} gpu:=true">
+  <xacro:macro name="OS1-32-N2" params="*origin parent:=base_link name:=ouster topic:=/ouster_points organize_cloud:=true hz:=10 lasers:=32 samples:=2048 collision_range:=0.5 min_range:=0.5 max_range:=90.0 noise:=0.00113 min_angle:=-${M_PI} max_angle:=${M_PI} gpu:=true">
     <joint name="${name}_base_mount_joint" type="fixed">
       <xacro:insert_block name="origin" />
@@ -68,6 +66,6 @@
                 <!-- <min_angle>-${30.67*M_PI/180.0}</min_angle> -->
                 <!-- <max_angle> ${10.67*M_PI/180.0}</max_angle> -->
-                <min_angle>-${45*M_PI/180.0}</min_angle>
-                <max_angle> ${45*M_PI/180.0}</max_angle>
+                <min_angle>-${22.5*M_PI/180.0}</min_angle>
+                <max_angle> ${22.5*M_PI/180.0}</max_angle>
               </vertical>
             </scan>
@@ -109,8 +107,6 @@
                 <samples>${lasers}</samples>
                 <resolution>1</resolution>
-                <!-- <min_angle>-${30.67*M_PI/180.0}</min_angle>
-                <max_angle> ${10.67*M_PI/180.0}</max_angle> -->
-                <min_angle>-${45*M_PI/180.0}</min_angle>
-                <max_angle> ${45*M_PI/180.0}</max_angle>
+                <min_angle>-${30.67*M_PI/180.0}</min_angle>
+                <max_angle> ${10.67*M_PI/180.0}</max_angle>
               </vertical>
             </scan>

File: ouster_description/urdf/OS2-32-N3.urdf.xacro (robot description, xacro)
@@ -1,6 +1,6 @@
 <?xml version="1.0"?>
-<robot xmlns:xacro="http://www.ros.org/wiki/xacro" name="OS1-128">
+<robot xmlns:xacro="http://www.ros.org/wiki/xacro" name="OS2-32-N3">
   <xacro:property name="M_PI" value="3.1415926535897931" />
-  <xacro:macro name="OS1-128" params="*origin parent:=base_link name:=ouster topic:=/ouster_points organize_cloud:=true hz:=10 lasers:=128 samples:=2048 collision_range:=0.5 min_range:=0.5 max_range:=90.0 noise:=0.008 min_angle:=-${M_PI} max_angle:=${M_PI} gpu:=true">
+  <xacro:macro name="OS2-32-N3" params="*origin parent:=base_link name:=ouster topic:=/ouster_points organize_cloud:=true hz:=10 lasers:=32 samples:=2048 collision_range:=0.5 min_range:=0.5 max_range:=90.0 noise:=0.0016 min_angle:=-${M_PI} max_angle:=${M_PI} gpu:=true">
     <joint name="${name}_base_mount_joint" type="fixed">
       <xacro:insert_block name="origin" />
@@ -66,6 +66,6 @@
                 <!-- <min_angle>-${30.67*M_PI/180.0}</min_angle> -->
                 <!-- <max_angle> ${10.67*M_PI/180.0}</max_angle> -->
-                <min_angle>-${22.5*M_PI/180.0}</min_angle>
-                <max_angle> ${22.5*M_PI/180.0}</max_angle>
+                <min_angle>-${11.25*M_PI/180.0}</min_angle>
+                <max_angle> ${11.25*M_PI/180.0}</max_angle>
               </vertical>
             </scan>

File: ouster_description/urdf/OS2-64-N1.urdf.xacro (robot description, xacro)
@@ -1,8 +1,6 @@
 <?xml version="1.0"?>
-<!-- <robot xmlns:xacro="http://www.ros.org/wiki/xacro" name="OS1-128"> -->
-<robot xmlns:xacro="http://www.ros.org/wiki/xacro" name="OSD-128">
+<robot xmlns:xacro="http://www.ros.org/wiki/xacro" name="OS2-64-N1">
   <xacro:property name="M_PI" value="3.1415926535897931" />
-  <!-- <xacro:macro name="OS1-128" params="*origin parent:=base_link name:=ouster topic:=/ouster_points organize_cloud:=true hz:=10 lasers:=128 samples:=2048 collision_range:=0.3 min_range:=0.5 max_range:=35.0 noise:=0.008 min_angle:=-${M_PI} max_angle:=${M_PI} gpu:=true"> -->
-  <xacro:macro name="OSD-128" params="*origin parent:=base_link name:=ouster topic:=/ouster_points organize_cloud:=true hz:=10 lasers:=128 samples:=2048 collision_range:=0.3 min_range:=0.5 max_range:=35.0 noise:=0.008 min_angle:=-${M_PI} max_angle:=${M_PI} gpu:=true">
+  <xacro:macro name="OS2-64-N1" params="*origin parent:=base_link name:=ouster topic:=/ouster_points organize_cloud:=true hz:=10 lasers:=64 samples:=2048 collision_range:=0.5 min_range:=0.5 max_range:=90.0 noise:=0.008 min_angle:=-${M_PI} max_angle:=${M_PI} gpu:=true">
     <joint name="${name}_base_mount_joint" type="fixed">
       <xacro:insert_block name="origin" />
@@ -68,6 +66,6 @@
                 <!-- <min_angle>-${30.67*M_PI/180.0}</min_angle> -->
                 <!-- <max_angle> ${10.67*M_PI/180.0}</max_angle> -->
-                <min_angle>-${0*M_PI/180.0}</min_angle>
-                <max_angle> ${85*M_PI/180.0}</max_angle>
+                <min_angle>-${11.25*M_PI/180.0}</min_angle>
+                <max_angle> ${11.25*M_PI/180.0}</max_angle>
               </vertical>
             </scan>
@@ -109,8 +107,6 @@
                 <samples>${lasers}</samples>
                 <resolution>1</resolution>
-                <!-- <min_angle>-${30.67*M_PI/180.0}</min_angle>
-                <max_angle> ${10.67*M_PI/180.0}</max_angle> -->
-                <min_angle>-${0*M_PI/180.0}</min_angle>
-                <max_angle> ${85*M_PI/180.0}</max_angle>
+                <min_angle>-${30.67*M_PI/180.0}</min_angle>
+                <max_angle> ${10.67*M_PI/180.0}</max_angle>
               </vertical>
             </scan>

File: ouster_description/urdf/OS2-64-N3.urdf.xacro (robot description, xacro)
@@ -1,8 +1,6 @@
 <?xml version="1.0"?>
-<!-- <robot xmlns:xacro="http://www.ros.org/wiki/xacro" name="OS1-128"> -->
-<robot xmlns:xacro="http://www.ros.org/wiki/xacro" name="OS2-128">
+<robot xmlns:xacro="http://www.ros.org/wiki/xacro" name="OS2-64-N3">
   <xacro:property name="M_PI" value="3.1415926535897931" />
-  <!-- <xacro:macro name="OS1-128" params="*origin parent:=base_link name:=ouster topic:=/ouster_points organize_cloud:=true hz:=10 lasers:=128 samples:=2048 collision_range:=0.8 min_range:=0.8 max_range:=200.0 noise:=0.008 min_angle:=-${M_PI} max_angle:=${M_PI} gpu:=true"> -->
-  <xacro:macro name="OS2-128" params="*origin parent:=base_link name:=ouster topic:=/ouster_points organize_cloud:=true hz:=10 lasers:=128 samples:=2048 collision_range:=0.8 min_range:=0.8 max_range:=200.0 noise:=0.008 min_angle:=-${M_PI} max_angle:=${M_PI} gpu:=true">
+  <xacro:macro name="OS2-64-N3" params="*origin parent:=base_link name:=ouster topic:=/ouster_points organize_cloud:=true hz:=10 lasers:=64 samples:=2048 collision_range:=0.5 min_range:=0.5 max_range:=90.0 noise:=0.0016 min_angle:=-${M_PI} max_angle:=${M_PI} gpu:=true">
     <joint name="${name}_base_mount_joint" type="fixed">
       <xacro:insert_block name="origin" />
@@ -20,5 +18,5 @@
       <visual>
         <geometry>
-          <mesh filename="package://ouster_description/meshes/OS2.dae" />
+          <mesh filename="package://ouster_description/meshes/OS1.dae" />
         </geometry>
       </visual>
@@ -44,5 +42,5 @@
         <origin xyz="0 0 -0.09081" rpy="0 0 0" />
         <geometry>
-          <mesh filename="package://ouster_description/meshes/OS2.dae" />
+          <mesh filename="package://ouster_description/meshes/OS1.dae" />
         </geometry>
       </visual>
