Commit message: updated husky xacro for fast lio

File: husky_description/urdf/husky.urdf.xacro (robot description, xacro)
@@ -70,12 +70,18 @@
   <xacro:arg name="laser_3d_secondary_rpy"        default="$(optenv HUSKY_LASER_3D_SECONDARY_RPY 0 0 -3.14159)" />
 <!-- Ouster LiDAR Primary and Secondary -->
-  <!-- No LiDAR = 0
-  OS1 = 1
-  OS2 = 2
-  OS0 = 3
-  -->
-  <xacro:arg name="OUSTER_OS"              default="$(optenv HUSKY_OUSTER 0)" />
-  <!-- <xacro:arg name="OUSTER_OS2_enabled"              default="$(optenv HUSKY_OUSTER_OS2_ENABLED 0)" /> -->
-  <!-- <xacro:arg name="OUSTER_OS0_enabled"              default="$(optenv HUSKY_OUSTER_OS0_ENABLED 0)" /> -->
+  <xacro:arg name="OUSTER_3D_enabled"              default="$(optenv HUSKY_OUSTER_3D_ENABLED 1)" />
+  <xacro:arg name="OUSTER_3D_topic"                default="$(optenv HUSKY_OUSTER_3D_TOPIC ouster_points)"/>
+  <xacro:arg name="OUSTER_3D_tower"                default="$(optenv HUSKY_OUSTER_3D_TOWER 1)"/>
+  <xacro:arg name="OUSTER_3D_prefix"               default="$(optenv HUSKY_OUSTER_3D_PREFIX )"/>
+  <xacro:arg name="OUSTER_3D_parent"               default="$(optenv HUSKY_OUSTER_3D_PARENT top_plate_link)"/>
+  <xacro:arg name="OUSTER_3D_xyz"                  default="$(optenv HUSKY_OUSTER_3D_XYZ 0 0 0)" />
+  <xacro:arg name="OUSTER_3D_rpy"                  default="$(optenv HUSKY_OUSTER_3D_RPY 0 0 0)" />
+  <xacro:arg name="OUSTER_3D_secondary_enabled"    default="$(optenv HUSKY_OUSTER_3D_SECONDARY_ENABLED 0)" />
+  <xacro:arg name="OUSTER_3D_secondary_topic"      default="$(optenv HUSKY_OUSTER_3D_SECONDARY_TOPIC ouster_secondary_points)"/>
+  <xacro:arg name="OUSTER_3D_secondary_tower"      default="$(optenv HUSKY_OUSTER_3D_SECONDARY_TOWER 1)"/>
+  <xacro:arg name="OUSTER_3D_secondary_prefix"     default="$(optenv HUSKY_OUSTER_3D_SECONDARY_PREFIX secondary_)"/>
+  <xacro:arg name="OUSTER_3D_secondary_parent"     default="$(optenv HUSKY_OUSTER_3D_SECONDARY_PARENT top_plate_link)"/>
+  <xacro:arg name="OUSTER_3D_secondary_xyz"        default="$(optenv HUSKY_OUSTER_3D_SECONDARY_XYZ 0 0 0)" />
+  <xacro:arg name="OUSTER_3D_secondary_rpy"        default="$(optenv HUSKY_OUSTER_3D_SECONDARY_RPY 0 0 -3.14159)" />
   <!-- Realsense Camera Primary and Secondary -->
   <xacro:arg name="realsense_enabled"             default="$(optenv HUSKY_REALSENSE_ENABLED 0)" />
@@ -99,4 +105,11 @@
   <xacro:arg name="blackfly_xyz"                      default="$(optenv HUSKY_BLACKFLY_XYZ 0 0 0)"/>
   <xacro:arg name="blackfly_rpy"                      default="$(optenv HUSKY_BLACKFLY_RPY 0 0 0)"/>
+  <xacro:arg name="blackfly_secondary_enabled"        default="$(optenv HUSKY_BLACKFLY_SECONDARY 0)"/>
+  <xacro:arg name="blackfly_secondary_mount_enabled"  default="$(optenv HUSKY_BLACKFLY_SECONDARY_MOUNT_ENABLED 1)"/>
+  <xacro:arg name="blackfly_secondary_mount_angle"    default="$(optenv HUSKY_BLACKFLY_SECONDARY_MOUNT_ANGLE 0)"/>
+  <xacro:arg name="blackfly_secondary_prefix"         default="$(optenv HUSKY_BLACKFLY_SECONDARY_PREFIX blackfly_secondary)"/>
+  <xacro:arg name="blackfly_secondary_parent"         default="$(optenv HUSKY_BLACKFLY_SECONDARY_PARENT top_plate_link)"/>
+  <xacro:arg name="blackfly_secondary_xyz"            default="$(optenv HUSKY_BLACKFLY_SECONDARY_XYZ 0 0 0)"/>
+  <xacro:arg name="blackfly_secondary_rpy"            default="$(optenv HUSKY_BLACKFLY_SECONDARY_RPY 0 0 0)"/>
   <!-- Bumper Extension -->
   <xacro:property name="husky_front_bumper_extend"  value="$(optenv HUSKY_FRONT_BUMPER_EXTEND 0)" />
@@ -121,8 +134,168 @@
   <xacro:include filename="$(find husky_description)/urdf/decorations.urdf.xacro" />
   <xacro:include filename="$(find husky_description)/urdf/wheel.urdf.xacro" />
-  <!-- <xacro:include filename="$(find ouster_description)/urdf/OS2-128.urdf.xacro"/>
-  <xacro:OS1-128 parent="top_plate_link" name="ouster">
-    <origin xyz="0 0 0.075" rpy="0 0 0" />
-  </xacro:OS1-128> -->
+  <xacro:arg name="OUSTER_OS"              default="$(optenv HUSKY_OUSTER 0)" />
+  <xacro:property name="model" value="$(arg OUSTER_OS)"/>
+  <xacro:if value="${model == 1}">
+    <xacro:include filename="$(find ouster_description)/urdf/OS1-128-N1.urdf.xacro"/>
+    <xacro:OS1-128-N1 parent="top_plate_link" name="ouster" topic="/ouster_points" organize_cloud="false" hz="10" samples="2048" gpu="true">
+    <origin xyz="0 0 0.1" rpy="0 0 0" />
+    </xacro:OS1-128-N1>
+  </xacro:if>
+  <xacro:if value="${model == 2}">
+    <xacro:include filename="$(find ouster_description)/urdf/OS2-128-N1.urdf.xacro"/>
+    <xacro:OS2-128-N1 parent="top_plate_link" name="ouster" topic="/ouster_points" organize_cloud="false" hz="10" samples="2048" gpu="true">
+    <origin xyz="0 0 0.1" rpy="0 0 0" />
+    </xacro:OS2-128-N1>
+  </xacro:if>
+  <xacro:if value="${model == 3}">
+    <xacro:include filename="$(find ouster_description)/urdf/OS0-128-N1.urdf.xacro"/>
+    <xacro:OS0-128-N1 parent="top_plate_link" name="ouster" topic="/ouster_points" organize_cloud="false" hz="10" samples="2048" gpu="true">
+    <origin xyz="0 0 0.1" rpy="0 0 0" />
+  </xacro:OS0-128-N1>
+  </xacro:if>
+  <xacro:if value="${model == 4}">
+    <xacro:include filename="$(find ouster_description)/urdf/OS1-64-N1.urdf.xacro"/>
+    <xacro:OS1-64-N1 parent="top_plate_link" name="ouster" topic="/ouster_points" organize_cloud="false" hz="10" samples="2048" gpu="true">
+    <origin xyz="0 0 0.1" rpy="0 0 0" />
+    </xacro:OS1-64-N1>
+  </xacro:if>
+  <xacro:if value="${model == 5}">
+    <xacro:include filename="$(find ouster_description)/urdf/OS2-64-N1.urdf.xacro"/>
+    <xacro:OS2-64-N1 parent="top_plate_link" name="ouster" topic="/ouster_points" organize_cloud="false" hz="10" samples="2048" gpu="true">
+    <origin xyz="0 0 0.1" rpy="0 0 0" />
+    </xacro:OS2-64-N1>
+  </xacro:if>
+  <xacro:if value="${model == 6}">
+    <xacro:include filename="$(find ouster_description)/urdf/OS0-64-N1.urdf.xacro"/>
+    <xacro:OS0-64-N1 parent="top_plate_link" name="ouster" topic="/ouster_points" organize_cloud="false" hz="10" samples="2048" gpu="true">
+    <origin xyz="0 0 0.1" rpy="0 0 0" />
+  </xacro:OS0-64-N1>
+  </xacro:if>
+  <xacro:if value="${model == 7}">
+    <xacro:include filename="$(find ouster_description)/urdf/OS1-32-N1.urdf.xacro"/>
+    <xacro:OS1-32-N1 parent="top_plate_link" name="ouster" topic="/ouster_points" organize_cloud="false" hz="10" samples="2048" gpu="true">
+    <origin xyz="0 0 0.1" rpy="0 0 0" />
+    </xacro:OS1-32-N1>
+  </xacro:if>
+  <xacro:if value="${model == 8}">
+    <xacro:include filename="$(find ouster_description)/urdf/OS2-32-N1.urdf.xacro"/>
+    <xacro:OS2-32-N1 parent="top_plate_link" name="ouster" topic="/ouster_points" organize_cloud="false" hz="10" samples="2048" gpu="true">
+    <origin xyz="0 0 0.1" rpy="0 0 0" />
+    </xacro:OS2-32-N1>
+  </xacro:if>
+  <xacro:if value="${model == 9}">
+    <xacro:include filename="$(find ouster_description)/urdf/OS0-32-N1.urdf.xacro"/>
+    <xacro:OS0-32-N1 parent="top_plate_link" name="ouster" topic="/ouster_points" organize_cloud="false" hz="10" samples="2048" gpu="true">
+    <origin xyz="0 0 0.1" rpy="0 0 0" />
+  </xacro:OS0-32-N1>
+  </xacro:if>
+  <xacro:if value="${model == 10}">
+    <xacro:include filename="$(find ouster_description)/urdf/OS1-128-N2.urdf.xacro"/>
+    <xacro:OS1-128-N2 parent="top_plate_link" name="ouster" topic="/ouster_points" organize_cloud="false" hz="10" samples="2048" gpu="true">
+    <origin xyz="0 0 0.1" rpy="0 0 0" />
+    </xacro:OS1-128-N2>
+  </xacro:if>
+  <xacro:if value="${model == 11}">
+    <xacro:include filename="$(find ouster_description)/urdf/OS2-128-N2.urdf.xacro"/>
+    <xacro:OS2-128-N2 parent="top_plate_link" name="ouster" topic="/ouster_points" organize_cloud="false" hz="10" samples="2048" gpu="true">
+    <origin xyz="0 0 0.1" rpy="0 0 0" />
+    </xacro:OS2-128-N2>
+  </xacro:if>
+  <xacro:if value="${model == 12}">
+    <xacro:include filename="$(find ouster_description)/urdf/OS0-128-N2.urdf.xacro"/>
+    <xacro:OS0-128-N2 parent="top_plate_link" name="ouster" topic="/ouster_points" organize_cloud="false" hz="10" samples="2048" gpu="true">
+    <origin xyz="0 0 0.1" rpy="0 0 0" />
+  </xacro:OS0-128-N2>
+  </xacro:if>
+  <xacro:if value="${model == 13}">
+    <xacro:include filename="$(find ouster_description)/urdf/OS1-64-N2.urdf.xacro"/>
+    <xacro:OS1-64-N2 parent="top_plate_link" name="ouster" topic="/ouster_points" organize_cloud="false" hz="10" samples="2048" gpu="true">
+    <origin xyz="0 0 0.1" rpy="0 0 0" />
+    </xacro:OS1-64-N2>
+  </xacro:if>
+  <xacro:if value="${model == 14}">
+    <xacro:include filename="$(find ouster_description)/urdf/OS2-64-N2.urdf.xacro"/>
+    <xacro:OS2-64-N2 parent="top_plate_link" name="ouster" topic="/ouster_points" organize_cloud="false" hz="10" samples="2048" gpu="true">
+    <origin xyz="0 0 0.1" rpy="0 0 0" />
+    </xacro:OS2-64-N2>
+  </xacro:if>
+  <xacro:if value="${model == 15}">
+    <xacro:include filename="$(find ouster_description)/urdf/OS0-64-N2.urdf.xacro"/>
+    <xacro:OS0-64-N2 parent="top_plate_link" name="ouster" topic="/ouster_points" organize_cloud="false" hz="10" samples="2048" gpu="true">
+    <origin xyz="0 0 0.1" rpy="0 0 0" />
+  </xacro:OS0-64-N2>
+  </xacro:if>
+  <xacro:if value="${model == 16}">
+    <xacro:include filename="$(find ouster_description)/urdf/OS1-32-N2.urdf.xacro"/>
+    <xacro:OS1-32-N2 parent="top_plate_link" name="ouster" topic="/ouster_points" organize_cloud="false" hz="10" samples="2048" gpu="true">
+    <origin xyz="0 0 0.1" rpy="0 0 0" />
+    </xacro:OS1-32-N2>
+  </xacro:if>
+  <xacro:if value="${model == 17}">
+    <xacro:include filename="$(find ouster_description)/urdf/OS2-32-N2.urdf.xacro"/>
+    <xacro:OS2-32-N2 parent="top_plate_link" name="ouster" topic="/ouster_points" organize_cloud="false" hz="10" samples="2048" gpu="true">
+    <origin xyz="0 0 0.1" rpy="0 0 0" />
+    </xacro:OS2-32-N2>
+  </xacro:if>
+  <xacro:if value="${model == 18}">
+    <xacro:include filename="$(find ouster_description)/urdf/OS0-32-N2.urdf.xacro"/>
+    <xacro:OS0-32-N2 parent="top_plate_link" name="ouster" topic="/ouster_points" organize_cloud="false" hz="10" samples="2048" gpu="true">
+    <origin xyz="0 0 0.1" rpy="0 0 0" />
+  </xacro:OS0-32-N2>
+  </xacro:if>
+  <xacro:if value="${model == 19}">
+    <xacro:include filename="$(find ouster_description)/urdf/OS1-128-N3.urdf.xacro"/>
+    <xacro:OS1-128-N3 parent="top_plate_link" name="ouster" topic="/ouster_points" organize_cloud="false" hz="10" samples="2048" gpu="true">
+    <origin xyz="0 0 0.1" rpy="0 0 0" />
+    </xacro:OS1-128-N3>
+  </xacro:if>
+  <xacro:if value="${model == 20}">
+    <xacro:include filename="$(find ouster_description)/urdf/OS2-128-N3.urdf.xacro"/>
+    <xacro:OS2-128-N3 parent="top_plate_link" name="ouster" topic="/ouster_points" organize_cloud="false" hz="10" samples="2048" gpu="true">
+    <origin xyz="0 0 0.1" rpy="0 0 0" />
+    </xacro:OS2-128-N3>
+  </xacro:if>
+  <xacro:if value="${model == 21}">
+    <xacro:include filename="$(find ouster_description)/urdf/OS0-128-N3.urdf.xacro"/>
+    <xacro:OS0-128-N3 parent="top_plate_link" name="ouster" topic="/ouster_points" organize_cloud="false" hz="10" samples="2048" gpu="true">
+    <origin xyz="0 0 0.1" rpy="0 0 0" />
+  </xacro:OS0-128-N3>
+  </xacro:if>
+  <xacro:if value="${model == 22}">
+    <xacro:include filename="$(find ouster_description)/urdf/OS1-64-N3.urdf.xacro"/>
+    <xacro:OS1-64-N3 parent="top_plate_link" name="ouster" topic="/ouster_points" organize_cloud="false" hz="10" samples="2048" gpu="true">
+    <origin xyz="0 0 0.1" rpy="0 0 0" />
+    </xacro:OS1-64-N3>
+  </xacro:if>
+  <xacro:if value="${model == 23}">
+    <xacro:include filename="$(find ouster_description)/urdf/OS2-64-N3.urdf.xacro"/>
+    <xacro:OS2-64-N3 parent="top_plate_link" name="ouster" topic="/ouster_points" organize_cloud="false" hz="10" samples="2048" gpu="true">
+    <origin xyz="0 0 0.1" rpy="0 0 0" />
+    </xacro:OS2-64-N3>
+  </xacro:if>
+  <xacro:if value="${model == 24}">
+    <xacro:include filename="$(find ouster_description)/urdf/OS0-64-N3.urdf.xacro"/>
+    <xacro:OS0-64-N3 parent="top_plate_link" name="ouster" topic="/ouster_points" organize_cloud="false" hz="10" samples="2048" gpu="true">
+    <origin xyz="0 0 0.1" rpy="0 0 0" />
+  </xacro:OS0-64-N3>
+  </xacro:if>
+  <xacro:if value="${model == 25}">
+    <xacro:include filename="$(find ouster_description)/urdf/OS1-32-N3.urdf.xacro"/>
+    <xacro:OS1-32-N3 parent="top_plate_link" name="ouster" topic="/ouster_points" organize_cloud="false" hz="10" samples="2048" gpu="true">
+    <origin xyz="0 0 0.1" rpy="0 0 0" />
+    </xacro:OS1-32-N3>
+  </xacro:if>
+  <xacro:if value="${model == 26}">
+    <xacro:include filename="$(find ouster_description)/urdf/OS2-32-N3.urdf.xacro"/>
+    <xacro:OS2-32-N3 parent="top_plate_link" name="ouster" topic="/ouster_points" organize_cloud="false" hz="10" samples="2048" gpu="true">
+    <origin xyz="0 0 0.1" rpy="0 0 0" />
+    </xacro:OS2-32-N3>
+  </xacro:if>
+  <xacro:if value="${model == 27}">
+    <xacro:include filename="$(find ouster_description)/urdf/OS0-32-N3.urdf.xacro"/>
+    <xacro:OS0-32-N3 parent="top_plate_link" name="ouster" topic="/ouster_points" organize_cloud="false" hz="10" samples="2048" gpu="true">
+    <origin xyz="0 0 0.1" rpy="0 0 0" />
+  </xacro:OS0-32-N3>
+  </xacro:if>
   <xacro:property name="M_PI" value="3.14159"/>
   <!-- Base Size -->
@@ -267,4 +440,12 @@
     </xacro:flir_blackfly_mount>
   </xacro:if>
+  <xacro:if value="$(arg blackfly_secondary_enabled)">
+    <xacro:flir_blackfly_mount prefix="$(arg blackfly_secondary_prefix)"
+                                parent="$(arg blackfly_secondary_parent)"
+                                mount_enabled="$(arg blackfly_secondary_mount_enabled)"
+                                mount_angle="$(arg blackfly_secondary_mount_angle)">
+      <origin xyz="$(arg blackfly_secondary_xyz)" rpy="$(arg blackfly_secondary_rpy)"/>
+    </xacro:flir_blackfly_mount>
+  </xacro:if>
   <!--
     Velodyne 3D LiDAR Primary and Secondary
@@ -295,171 +476,30 @@
   </xacro:if>
   <!--
-    Ouster OS LiDAR
+    Ouster 3D LiDAR Primary and Secondary
   -->
-  <xacro:property name="model" value="$(arg OUSTER_OS)"/>
-  <xacro:if value="${model == 1}">
-    <xacro:include filename="$(find ouster_description)/urdf/OS1-128-N1.urdf.xacro"/>
-    <xacro:OS1-128-N1 parent="top_plate_link" name="ouster">
-      <origin xyz="0 0 0.075" rpy="0 0 0" />
-    </xacro:OS1-128-N1>
-  </xacro:if>
-  <xacro:if value="${model == 2}">
-    <xacro:include filename="$(find ouster_description)/urdf/OS2-128-N1.urdf.xacro"/>
-    <xacro:OS2-128-N1 parent="top_plate_link" name="ouster">
-      <origin xyz="0 0 0.075" rpy="0 0 0" />
-    </xacro:OS2-128-N1>
-  </xacro:if>
-  <xacro:if value="${model == 3}">
-    <xacro:include filename="$(find ouster_description)/urdf/OS0-128-N1.urdf.xacro"/>
-    <xacro:OS0-128-N1 parent="top_plate_link" name="ouster">
-      <origin xyz="0 0 0.075" rpy="0 0 0" />
-    </xacro:OS0-128-N1>
-  </xacro:if>
-  <xacro:if value="${model == 4}">
-    <xacro:include filename="$(find ouster_description)/urdf/OS1-64-N1.urdf.xacro"/>
-    <xacro:OS1-64-N1 parent="top_plate_link" name="ouster">
-      <origin xyz="0 0 0.075" rpy="0 0 0" />
-    </xacro:OS1-64-N1>
-  </xacro:if>
-  <xacro:if value="${model == 5}">
-    <xacro:include filename="$(find ouster_description)/urdf/OS2-64-N1.urdf.xacro"/>
-    <xacro:OS2-64-N1 parent="top_plate_link" name="ouster">
-      <origin xyz="0 0 0.075" rpy="0 0 0" />
-    </xacro:OS2-64-N1>
-  </xacro:if>
-  <xacro:if value="${model == 6}">
-    <xacro:include filename="$(find ouster_description)/urdf/OS0-64-N1.urdf.xacro"/>
-    <xacro:OS0-64-N1 parent="top_plate_link" name="ouster">
-      <origin xyz="0 0 0.075" rpy="0 0 0" />
-    </xacro:OS0-64-N1>
-  </xacro:if>
-  <xacro:if value="${model == 7}">
-    <xacro:include filename="$(find ouster_description)/urdf/OS1-32-N1.urdf.xacro"/>
-    <xacro:OS1-32-N1 parent="top_plate_link" name="ouster">
-      <origin xyz="0 0 0.075" rpy="0 0 0" />
-    </xacro:OS1-32-N1>
-  </xacro:if>
-  <xacro:if value="${model == 8}">
-    <xacro:include filename="$(find ouster_description)/urdf/OS2-32-N1.urdf.xacro"/>
-    <xacro:OS2-32-N1 parent="top_plate_link" name="ouster">
-      <origin xyz="0 0 0.075" rpy="0 0 0" />
-    </xacro:OS2-32-N1>
-  </xacro:if>
-  <xacro:if value="${model == 9}">
-    <xacro:include filename="$(find ouster_description)/urdf/OS0-32-N1.urdf.xacro"/>
-    <xacro:OS0-32-N1 parent="top_plate_link" name="ouster">
-      <origin xyz="0 0 0.075" rpy="0 0 0" />
-    </xacro:OS0-32-N1>
-  </xacro:if>
-  <xacro:property name="model" value="$(arg OUSTER_OS)"/>
-  <xacro:if value="${model == 10}">
-    <xacro:include filename="$(find ouster_description)/urdf/OS1-128-N2.urdf.xacro"/>
-    <xacro:OS1-128-N2 parent="top_plate_link" name="ouster">
-      <origin xyz="0 0 0.075" rpy="0 0 0" />
-    </xacro:OS1-128-N2>
-  </xacro:if>
-  <xacro:if value="${model == 11}">
-    <xacro:include filename="$(find ouster_description)/urdf/OS2-128-N2.urdf.xacro"/>
-    <xacro:OS2-128-N2 parent="top_plate_link" name="ouster">
-      <origin xyz="0 0 0.075" rpy="0 0 0" />
-    </xacro:OS2-128-N2>
-  </xacro:if>
-  <xacro:if value="${model == 12}">
-    <xacro:include filename="$(find ouster_description)/urdf/OS0-128-N2.urdf.xacro"/>
-    <xacro:OS0-128-N2 parent="top_plate_link" name="ouster">
-      <origin xyz="0 0 0.075" rpy="0 0 0" />
-    </xacro:OS0-128-N2>
-  </xacro:if>
-  <xacro:if value="${model == 13}">
-    <xacro:include filename="$(find ouster_description)/urdf/OS1-64-N2.urdf.xacro"/>
-    <xacro:OS1-64-N2 parent="top_plate_link" name="ouster">
-      <origin xyz="0 0 0.075" rpy="0 0 0" />
-    </xacro:OS1-64-N2>
-  </xacro:if>
-  <xacro:if value="${model == 14}">
-    <xacro:include filename="$(find ouster_description)/urdf/OS2-64-N2.urdf.xacro"/>
-    <xacro:OS2-64-N2 parent="top_plate_link" name="ouster">
-      <origin xyz="0 0 0.075" rpy="0 0 0" />
-    </xacro:OS2-64-N2>
-  </xacro:if>
-  <xacro:if value="${model == 15}">
-    <xacro:include filename="$(find ouster_description)/urdf/OS0-64-N2.urdf.xacro"/>
-    <xacro:OS0-64-N2 parent="top_plate_link" name="ouster">
-      <origin xyz="0 0 0.075" rpy="0 0 0" />
-    </xacro:OS0-64-N2>
-  </xacro:if>
-  <xacro:if value="${model == 16}">
-    <xacro:include filename="$(find ouster_description)/urdf/OS1-32-N2.urdf.xacro"/>
-    <xacro:OS1-32-N2 parent="top_plate_link" name="ouster">
-      <origin xyz="0 0 0.075" rpy="0 0 0" />
-    </xacro:OS1-32-N2>
-  </xacro:if>
-  <xacro:if value="${model == 17}">
-    <xacro:include filename="$(find ouster_description)/urdf/OS2-32-N2.urdf.xacro"/>
-    <xacro:OS2-32-N2 parent="top_plate_link" name="ouster">
-      <origin xyz="0 0 0.075" rpy="0 0 0" />
-    </xacro:OS2-32-N2>
-  </xacro:if>
-  <xacro:if value="${model == 18}">
-    <xacro:include filename="$(find ouster_description)/urdf/OS0-32-N2.urdf.xacro"/>
-    <xacro:OS0-32-N2 parent="top_plate_link" name="ouster">
-      <origin xyz="0 0 0.075" rpy="0 0 0" />
-    </xacro:OS0-32-N2>
-  </xacro:if>
-  <xacro:property name="model" value="$(arg OUSTER_OS)"/>
-  <xacro:if value="${model == 19}">
-    <xacro:include filename="$(find ouster_description)/urdf/OS1-128-N3.urdf.xacro"/>
-    <xacro:OS1-128-N3 parent="top_plate_link" name="ouster">
-      <origin xyz="0 0 0.075" rpy="0 0 0" />
-    </xacro:OS1-128-N3>
-  </xacro:if>
-  <xacro:if value="${model == 20}">
-    <xacro:include filename="$(find ouster_description)/urdf/OS2-128-N3.urdf.xacro"/>
-    <xacro:OS2-128-N3 parent="top_plate_link" name="ouster">
-      <origin xyz="0 0 0.075" rpy="0 0 0" />
-    </xacro:OS2-128-N3>
-  </xacro:if>
-  <xacro:if value="${model == 21}">
-    <xacro:include filename="$(find ouster_description)/urdf/OS0-128-N3.urdf.xacro"/>
-    <xacro:OS0-128-N3 parent="top_plate_link" name="ouster">
-      <origin xyz="0 0 0.075" rpy="0 0 0" />
-    </xacro:OS0-128-N3>
-  </xacro:if>
-  <xacro:if value="${model == 22}">
-    <xacro:include filename="$(find ouster_description)/urdf/OS1-64-N3.urdf.xacro"/>
-    <xacro:OS1-64-N3 parent="top_plate_link" name="ouster">
-      <origin xyz="0 0 0.075" rpy="0 0 0" />
-    </xacro:OS1-64-N3>
-  </xacro:if>
-  <xacro:if value="${model == 23}">
-    <xacro:include filename="$(find ouster_description)/urdf/OS2-64-N3.urdf.xacro"/>
-    <xacro:OS2-64-N3 parent="top_plate_link" name="ouster">
-      <origin xyz="0 0 0.075" rpy="0 0 0" />
-    </xacro:OS2-64-N3>
-  </xacro:if>
-  <xacro:if value="${model == 24}">
-    <xacro:include filename="$(find ouster_description)/urdf/OS0-64-N3.urdf.xacro"/>
-    <xacro:OS0-64-N3 parent="top_plate_link" name="ouster">
-      <origin xyz="0 0 0.075" rpy="0 0 0" />
-    </xacro:OS0-64-N3>
-  </xacro:if>
-  <xacro:if value="${model == 25}">
-    <xacro:include filename="$(find ouster_description)/urdf/OS1-32-N3.urdf.xacro"/>
-    <xacro:OS1-32-N3 parent="top_plate_link" name="ouster">
-      <origin xyz="0 0 0.075" rpy="0 0 0" />
-    </xacro:OS1-32-N3>
-  </xacro:if>
-  <xacro:if value="${model == 26}">
-    <xacro:include filename="$(find ouster_description)/urdf/OS2-32-N3.urdf.xacro"/>
-    <xacro:OS2-32-N3 parent="top_plate_link" name="ouster">
-      <origin xyz="0 0 0.075" rpy="0 0 0" />
-    </xacro:OS2-32-N3>
-  </xacro:if>
-  <xacro:if value="${model == 27}">
-    <xacro:include filename="$(find ouster_description)/urdf/OS0-32-N3.urdf.xacro"/>
-    <xacro:OS0-32-N3 parent="top_plate_link" name="ouster">
-      <origin xyz="0 0 0.075" rpy="0 0 0" />
-    </xacro:OS0-32-N3>
-  </xacro:if>
+  <!-- <xacro:if value="$(arg OUSTER_3D_enabled)">
+    <xacro:if value="$(arg OUSTER_3D_tower)">
+      <xacro:vlp16_mount prefix="$(arg OUSTER_3D_prefix)" parent_link="$(arg OUSTER_3D_parent)" topic="$(arg OUSTER_3D_topic)">
+        <origin xyz="$(arg OUSTER_3D_xyz)" rpy="$(arg OUSTER_3D_rpy)" />
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
File: ouster_description/urdf/OS1-128-N1.urdf.xacro (robot description, xacro)
@@ -2,5 +2,5 @@
 <robot xmlns:xacro="http://www.ros.org/wiki/xacro" name="OS1-128-N1">
   <xacro:property name="M_PI" value="3.1415926535897931" />
-  <xacro:macro name="OS1-128-N1" params="*origin parent:=base_link name:=ouster topic:=/ouster_points organize_cloud:=true hz:=10 lasers:=128 samples:=2048 collision_range:=0.5 min_range:=0.5 max_range:=90.0 noise:=0.008 min_angle:=-${M_PI} max_angle:=${M_PI} gpu:=true">
+  <xacro:macro name="OS1-128-N1" params="*origin parent:=base_link name:=ouster topic:=/ouster_points organize_cloud:=true hz:=10 lasers:=128 samples:=2048 collision_range:=0.3 min_range:=0.3 max_range:=100.0 noise:=0.008 min_angle:=-${M_PI} max_angle:=${M_PI} gpu:=false">
     <joint name="${name}_base_mount_joint" type="fixed">
       <xacro:insert_block name="origin" />

File: ouster_description/urdf/OS2-32-N1.urdf.xacro (robot description, xacro)
@@ -1,3 +1,3 @@
-w<?xml version="1.0"?>
+<?xml version="1.0"?>
 <robot xmlns:xacro="http://www.ros.org/wiki/xacro" name="OS2-32-N1">
   <xacro:property name="M_PI" value="3.1415926535897931" />
